Commit message: Imported upstream version '1.0.4' of 'upstream'

File: clober_description/urdf/clober.gazebo.xacro (robot description, xacro)
@@ -3,8 +3,8 @@
   <xacro:arg name="laser_visual" default="true"/>
   <xacro:arg name="imu_visual"   default="false"/>
-  <gazebo reference="base_link">
+  <gazebo reference="$(arg prefix)base_link">
     <material>Gazebo/White</material>
   </gazebo>
-  <gazebo reference="wheel_left_link">
+  <gazebo reference="$(arg prefix)wheel_left_link">
     <mu1>0.1</mu1>
     <mu2>0.1</mu2>
@@ -16,5 +16,5 @@
     <material>Gazebo/FlatBlack</material>
   </gazebo>
-  <gazebo reference="wheel_right_link">
+  <gazebo reference="$(arg prefix)wheel_right_link">
     <mu1>0.1</mu1>
     <mu2>0.1</mu2>
@@ -26,5 +26,5 @@
     <material>Gazebo/FlatBlack</material>
   </gazebo>
-  <gazebo reference="caster_link1">
+  <gazebo reference="$(arg prefix)caster_link1">
     <mu1>0.05</mu1>
     <mu2>0.05</mu2>
@@ -36,5 +36,5 @@
     <material>Gazebo/FlatBlack</material>
   </gazebo>
-  <gazebo reference="caster_link2">
+  <gazebo reference="$(arg prefix)caster_link2">
     <mu1>0.05</mu1>
     <mu2>0.05</mu2>
@@ -46,5 +46,5 @@
     <material>Gazebo/FlatBlack</material>
   </gazebo>
-  <gazebo reference="caster_link3">
+  <gazebo reference="$(arg prefix)caster_link3">
     <mu1>0.05</mu1>
     <mu2>0.05</mu2>
@@ -56,5 +56,5 @@
     <material>Gazebo/FlatBlack</material>
   </gazebo>
-  <gazebo reference="caster_link4">
+  <gazebo reference="$(arg prefix)caster_link4">
     <mu1>0.05</mu1>
     <mu2>0.05</mu2>
@@ -66,5 +66,5 @@
     <material>Gazebo/FlatBlack</material>
   </gazebo>
-  <gazebo reference="imu_link">
+  <gazebo reference="$(arg prefix)imu_link">
     <sensor type="imu" name="imu">
       <always_on>true</always_on>
@@ -77,8 +77,8 @@
       <commandTopic>cmd_vel</commandTopic>
       <odometryTopic>odom</odometryTopic>
-      <odometryFrame>odom</odometryFrame>
+      <odometryFrame>$(arg prefix)odom</odometryFrame>
       <odometrySource>world</odometrySource>
       <publishOdomTF>true</publishOdomTF>
-      <robotBaseFrame>base_footprint</robotBaseFrame>
+      <robotBaseFrame>$(arg prefix)base_footprint</robotBaseFrame>
       <publishWheelTF>false</publishWheelTF>
       <publishTf>true</publishTf>
@@ -86,6 +86,6 @@
       <legacyMode>false</legacyMode>
       <updateRate>30</updateRate>
-      <leftJoint>wheel_left_joint</leftJoint>
-      <rightJoint>wheel_right_joint</rightJoint>
+      <leftJoint>$(arg prefix)wheel_left_joint</leftJoint>
+      <rightJoint>$(arg prefix)wheel_right_joint</rightJoint>
       <wheelSeparation>0.310</wheelSeparation>
       <wheelDiameter>0.17</wheelDiameter>
@@ -98,6 +98,6 @@
     <plugin name="imu_plugin" filename="libgazebo_ros_imu.so">
       <alwaysOn>true</alwaysOn>
-      <bodyName>imu_link</bodyName>
-      <frameName>imu_link</frameName>
+      <bodyName>$(arg prefix)imu_link</bodyName>
+      <frameName>$(arg prefix)imu_link</frameName>
       <topicName>imu</topicName>
       <serviceName>imu_service</serviceName>
@@ -123,5 +123,5 @@
     </plugin>
   </gazebo>
-  <gazebo reference="base_scan">
+  <gazebo reference="$(arg prefix)base_scan">
     <material>Gazebo/FlatBlack</material>
     <sensor type="ray" name="lds_lfcd_sensor">
@@ -151,5 +151,5 @@
       <plugin name="gazebo_ros_lds_lfcd_controller" filename="libgazebo_ros_laser.so">
         <topicName>scan</topicName>
-        <frameName>base_scan</frameName>
+        <frameName>$(arg prefix)base_scan</frameName>
       </plugin>
     </sensor>

File: clober_description/urdf/clober.urdf.xacro (robot description, xacro)
@@ -7,11 +7,11 @@
     <xacro:include filename="$(find clober_description)/urdf/clober.gazebo.xacro"/>
     <xacro:property name="PI" value="3.1415926535897931"/>
-    <link name="base_footprint"/>
-    <joint name="base_joint" type="fixed">
-        <parent link="base_footprint"/>
-        <child link="base_link"/>
+    <link name="$(arg prefix)base_footprint"/>
+    <joint name="$(arg prefix)base_joint" type="fixed">
+        <parent link="$(arg prefix)base_footprint"/>
+        <child link="$(arg prefix)base_link"/>
         <origin xyz="0.0 0.0 0.020" rpy="0 0 0"/>
     </joint>
-    <link name="base_link">
+    <link name="$(arg prefix)base_link">
         <visual>
             <origin xyz="0 0 0" rpy="0 0 ${PI/2}"/>
@@ -38,11 +38,11 @@
         </inertial>
     </link>
-    <joint name="wheel_left_joint" type="continuous">
-        <parent link="base_link"/>
-        <child link="wheel_left_link"/>
+    <joint name="$(arg prefix)wheel_left_joint" type="continuous">
+        <parent link="$(arg prefix)base_link"/>
+        <child link="$(arg prefix)wheel_left_link"/>
         <origin xyz="0.0018 0.1558 0.02" rpy="0 0 0"/>
         <axis xyz="0 1 0" rpy="0 0 0"/>
     </joint>
-    <link name="wheel_left_link">
+    <link name="$(arg prefix)wheel_left_link">
         <visual>
             <origin xyz="0 0 0" rpy="0 0 -${PI/2}"/>
@@ -69,11 +69,11 @@
         </inertial>
     </link>
-    <joint name="wheel_right_joint" type="continuous">
-        <parent link="base_link"/>
-        <child link="wheel_right_link"/>
+    <joint name="$(arg prefix)wheel_right_joint" type="continuous">
+        <parent link="$(arg prefix)base_link"/>
+        <child link="$(arg prefix)wheel_right_link"/>
         <origin xyz="0.0018 -0.1558 0.02" rpy="0 0 0"/>
         <axis xyz="0 1 0" rpy="0 0 0"/>
     </joint>
-    <link name="wheel_right_link">
+    <link name="$(arg prefix)wheel_right_link">
         <visual>
             <origin xyz="0 0 0" rpy="0 0 ${PI/2}"/>
@@ -100,105 +100,105 @@
         </inertial>
     </link>
-    <joint name="caster_joint1" type="continuous">
-        <parent link="base_link"/>
-        <child link="caster_link1"/>
+    <joint name="$(arg prefix)caster_joint1" type="continuous">
+        <parent link="$(arg prefix)base_link"/>
+        <child link="$(arg prefix)caster_link1"/>
         <origin xyz="0.11 0.13 -0.04" rpy="${PI/2} 0 0"/>
         <axis xyz="0 0 1" rpy="0 0 0"/>
     </joint>
-    <link name="caster_link1">
-        <collision>
-            <origin xyz="0 0 0" rpy="0 0 0"/>
-            <geometry>
-                <cylinder length="0.02" radius="0.025"/>
-            </geometry>
-        </collision>
-        <inertial>
-            <origin xyz="0 0 0"/>
-            <mass value="0.005"/>
-            <inertia ixx="0.001" ixy="0.0" ixz="0.0" iyy="0.001" iyz="0.0" izz="0.001"/>
-        </inertial>
-    </link>
-    <joint name="caster_joint2" type="continuous">
-        <parent link="base_link"/>
-        <child link="caster_link2"/>
+    <link name="$(arg prefix)caster_link1">
+        <collision>
+            <origin xyz="0 0 0" rpy="0 0 0"/>
+            <geometry>
+                <cylinder length="0.02" radius="0.025"/>
+            </geometry>
+        </collision>
+        <inertial>
+            <origin xyz="0 0 0"/>
+            <mass value="0.005"/>
+            <inertia ixx="0.001" ixy="0.0" ixz="0.0" iyy="0.001" iyz="0.0" izz="0.001"/>
+        </inertial>
+    </link>
+    <joint name="$(arg prefix)caster_joint2" type="continuous">
+        <parent link="$(arg prefix)base_link"/>
+        <child link="$(arg prefix)caster_link2"/>
         <origin xyz="-0.11 0.13 -0.04" rpy="${PI/2} 0 0"/>
         <axis xyz="0 0 1" rpy="0 0 0"/>
     </joint>
-    <link name="caster_link2">
-        <collision>
-            <origin xyz="0 0 0" rpy="0 0 0"/>
-            <geometry>
-                <cylinder length="0.02" radius="0.025"/>
-            </geometry>
-        </collision>
-        <inertial>
-            <origin xyz="0 0 0"/>
-            <mass value="0.005"/>
-            <inertia ixx="0.001" ixy="0.0" ixz="0.0" iyy="0.001" iyz="0.0" izz="0.001"/>
-        </inertial>
-    </link>
-    <joint name="caster_joint3" type="continuous">
-        <parent link="base_link"/>
-        <child link="caster_link3"/>
+    <link name="$(arg prefix)caster_link2">
+        <collision>
+            <origin xyz="0 0 0" rpy="0 0 0"/>
+            <geometry>
+                <cylinder length="0.02" radius="0.025"/>
+            </geometry>
+        </collision>
+        <inertial>
+            <origin xyz="0 0 0"/>
+            <mass value="0.005"/>
+            <inertia ixx="0.001" ixy="0.0" ixz="0.0" iyy="0.001" iyz="0.0" izz="0.001"/>
+        </inertial>
+    </link>
+    <joint name="$(arg prefix)caster_joint3" type="continuous">
+        <parent link="$(arg prefix)base_link"/>
+        <child link="$(arg prefix)caster_link3"/>
         <origin xyz="0.11 -0.13 -0.04" rpy="${PI/2} 0 0"/>
         <axis xyz="0 0 1" rpy="0 0 0"/>
     </joint>
-    <link name="caster_link3">
-        <collision>
-            <origin xyz="0 0 0" rpy="0 0 0"/>
-            <geometry>
-                <cylinder length="0.02" radius="0.025"/>
-            </geometry>
-        </collision>
-        <inertial>
-            <origin xyz="0 0 0"/>
-            <mass value="0.005"/>
-            <inertia ixx="0.001" ixy="0.0" ixz="0.0" iyy="0.001" iyz="0.0" izz="0.001"/>
-        </inertial>
-    </link>
-    <joint name="caster_joint4" type="continuous">
-        <parent link="base_link"/>
-        <child link="caster_link4"/>
+    <link name="$(arg prefix)caster_link3">
+        <collision>
+            <origin xyz="0 0 0" rpy="0 0 0"/>
+            <geometry>
+                <cylinder length="0.02" radius="0.025"/>
+            </geometry>
+        </collision>
+        <inertial>
+            <origin xyz="0 0 0"/>
+            <mass value="0.005"/>
+            <inertia ixx="0.001" ixy="0.0" ixz="0.0" iyy="0.001" iyz="0.0" izz="0.001"/>
+        </inertial>
+    </link>
+    <joint name="$(arg prefix)caster_joint4" type="continuous">
+        <parent link="$(arg prefix)base_link"/>
+        <child link="$(arg prefix)caster_link4"/>
         <origin xyz="-0.11 -0.13 -0.04" rpy="${PI/2} 0 0"/>
         <axis xyz="0 0 1" rpy="0 0 0"/>
     </joint>
-    <link name="caster_link4">
-        <collision>
-            <origin xyz="0 0 0" rpy="0 0 0"/>
-            <geometry>
-                <cylinder length="0.02" radius="0.025"/>
-            </geometry>
-        </collision>
-        <inertial>
-            <origin xyz="0 0 0"/>
-            <mass value="0.005"/>
-            <inertia ixx="0.001" ixy="0.0" ixz="0.0" iyy="0.001" iyz="0.0" izz="0.001"/>
-        </inertial>
-    </link>
-    <joint name="imu_joint" type="fixed">
-        <parent link="base_link"/>
-        <child link="imu_link"/>
+    <link name="$(arg prefix)caster_link4">
+        <collision>
+            <origin xyz="0 0 0" rpy="0 0 0"/>
+            <geometry>
+                <cylinder length="0.02" radius="0.025"/>
+            </geometry>
+        </collision>
+        <inertial>
+            <origin xyz="0 0 0"/>
+            <mass value="0.005"/>
+            <inertia ixx="0.001" ixy="0.0" ixz="0.0" iyy="0.001" iyz="0.0" izz="0.001"/>
+        </inertial>
+    </link>
+    <joint name="$(arg prefix)imu_joint" type="fixed">
+        <parent link="$(arg prefix)base_link"/>
+        <child link="$(arg prefix)imu_link"/>
         <origin xyz="0.0605 0 0.0923" rpy="0 0 0"/>
     </joint>
-    <link name="imu_link"/>
-    <joint name="left_ultrasonic_joint" type="fixed">
-        <parent link="base_link"/>
-        <child link="left_ultrasonic"/>
+    <link name="$(arg prefix)imu_link"/>
+    <joint name="$(arg prefix)left_ultrasonic_joint" type="fixed">
+        <parent link="$(arg prefix)base_link"/>
+        <child link="$(arg prefix)left_ultrasonic"/>
         <origin xyz="0.18164 0.09679 0.08396" rpy="0 0 0"/>
     </joint>
-    <link name="left_ultrasonic"/>
-    <joint name="right_ultrasonic_joint" type="fixed">
-        <parent link="base_link"/>
-        <child link="right_ultrasonic"/>
+    <link name="$(arg prefix)left_ultrasonic"/>
+    <joint name="$(arg prefix)right_ultrasonic_joint" type="fixed">
+        <parent link="$(arg prefix)base_link"/>
+        <child link="$(arg prefix)right_ultrasonic"/>
         <origin xyz="0.18164 -0.09679 0.08396" rpy="0 0 0"/>
     </joint>
-    <link name="right_ultrasonic"/>
-    <joint name="base_scan_joint" type="fixed">
-        <parent link="base_link"/>
-        <child link="base_scan"/>
+    <link name="$(arg prefix)right_ultrasonic"/>
+    <joint name="$(arg prefix)base_scan_joint" type="fixed">
+        <parent link="$(arg prefix)base_link"/>
+        <child link="$(arg prefix)base_scan"/>
         <origin xyz="0.159 0 0.16" rpy="${PI} 0 0"/>
     </joint>
     <!-- <origin xyz="0.21 0 0.16" rpy="${PI} 0 0"/> -->
-    <link name="base_scan">
+    <link name="$(arg prefix)base_scan">
       <visual>
           <origin xyz="0 0 0"    rpy="0 0 0"/>
@@ -210,5 +210,5 @@
     <!-- <xacro:sensor_tim571 parent="base_link"> <origin xyz="0.159 0 0.2265"
     rpy="${PI} 0 0"/> </xacro:sensor_tim571> -->
-    <xacro:sensor_d435 parent="base_link" name="camera">
+    <xacro:sensor_d435 parent="$(arg prefix)base_link" name="$(arg prefix)camera">
         <origin xyz="0.17573 0 0.06791" rpy="0 -${PI/12} 0"/>
     </xacro:sensor_d435>
